File: kicad/clock_gen.kicad_pcb (KiCad board)
At the start: 2 copper layers, 20 parts, among them J1 Programming, SW1 Rotary_Encoder, SW2 Rotary_Encoder, U1 MachXO2-1200-QFN32, U2 LM3480-3.3, U3 74HCT541, X1 DSC1001AE5-001.2000

Commit message: Finished PCB
Parts:
- added C12: 1uF, Capacitor_SMD:C_0603_1608Metric, F.Cu at (93.8, 126.3)
- added D1: IN-S63AT5G, LED_SMD:LED_0603_1608Metric, F.Cu at (100.1, 124.0)
- added D2: LTST-C190KRKT, LED_SMD:LED_0603_1608Metric, F.Cu at (82.2, 140.0)
- added J2: buf_output, Connector_PinHeader_1.27mm:PinHeader_1x08_P1.27mm_Vertical, F.Cu at (108.6, 128.5)
- added J3: Power, Connector_PinHeader_1.27mm:PinHeader_1x03_P1.27mm_Vertical, F.Cu at (81.7, 123.2)
- added J4: CLRN, Connector_PinHeader_1.27mm:PinHeader_1x01_P1.27mm_Vertical, F.Cu at (89.1, 128.1)
- added LOGO1: Logo_Open_Hardware_Large, logo:clk, B.Cu at (95.2, 132.0)
- added R2: 1k, Resistor_SMD:R_0603_1608Metric, F.Cu at (96.9, 124.0)
- added R3: 1k, Resistor_SMD:R_0603_1608Metric, F.Cu at (82.2, 142.9)
- SW1, SW2: footprint Potentiometer_THT:Potentiometer_Bourns_PTV09A-2_Single_Horizontal -> Connector_PinHeader_1.27mm:PinHeader_1x03_P1.27mm_Vertical
- U2: value LM3480-3.3 -> MIC5504-3.3YM5; footprint Package_TO_SOT_SMD:SOT-23 -> Package_TO_SOT_SMD:SOT-23-5
- moved SW2 14.5 mm to (81.7, 133.3), turned to 0 degrees
- moved SW1 12.3 mm to (81.7, 128.3), turned to 0 degrees
- moved J1 9.28 mm to (92.4, 142.6)
- moved U2 7.74 mm to (91.2, 126.0), turned to 270 degrees
- moved C1 6.05 mm to (84.4, 123.9), turned to 270 degrees
- moved U3 4.05 mm to (101.6, 131.7)
- moved C2 3.99 mm to (85.9, 123.9), turned to 270 degrees
- moved X1 3.80 mm to (86.8, 140.9)
- moved C3 1.94 mm to (87.3, 123.9), turned to 270 degrees
- moved L1 1.72 mm to (89.4, 123.1), turned to 180 degrees
- moved C6 0.30 mm to (92.2, 137.2)
- moved R1 0.30 mm to (92.2, 138.7)
Connections:
- net EXT3v3 renamed EXT5v
- net PT12D/SDA renamed Net-(U1-Pad27)
- net PT15C/JTAGENB renamed Net-(U1-Pad26)
- net PT15D/PROGRAMN renamed Net-(U1-Pad25)
- L1 pad 1: +3V3 -> +5V
- SW1 pad 1: (no net) -> E1A
- SW1 pad 2: (no net) -> GND
- SW1 pad 3: (no net) -> E1B
- SW2 pad 1: (no net) -> E2A
- SW2 pad 2: (no net) -> GND
- SW2 pad 3: (no net) -> E2B
- U1 pad 10: PB6D/MISO -> clk_60k
- U1 pad 11: PB9A -> clk_80k
- U1 pad 12: PB9B -> clk_100k
- U1 pad 13: PB11A -> clk_1M2
- U1 pad 14: PB11B -> clrn
- U1 pad 16: PB20C/SN -> E1A
- U1 pad 17: PB20D/MOSI -> E1B
- U1 pad 20: PR5D -> E2A
- U1 pad 21: PR5C -> E2B
- U1 pad 23: PT17D/DONE -> led
- U1 pad 28: PT12C/SCL -> pin1
- U1 pad 4: PL9A -> pin2
- U1 pad 5: PL9B -> Blanking
- U1 pad 8: PB4C/CS -> clk_20k
- U1 pad 9: PB6C/SCLK -> clk_40k
- U2 pad 1: Net-(U2-Pad1) -> +5V
- U2 pad 2: Net-(U2-Pad2) -> GND
- U2 pad 3: Net-(U2-Pad3) -> +5V
- U3 pad 1: Net-(U3-Pad1) -> GND
- U3 pad 10: Net-(U3-Pad10) -> GND
- U3 pad 19: Net-(U3-Pad19) -> GND
- U3 pad 2: Net-(U3-Pad2) -> clk_100k
- U3 pad 20: Net-(U3-Pad20) -> +5V
- U3 pad 3: Net-(U3-Pad3) -> clk_80k
- U3 pad 4: Net-(U3-Pad4) -> clk_60k
- U3 pad 5: Net-(U3-Pad5) -> clk_40k
- U3 pad 6: Net-(U3-Pad6) -> clk_20k
- U3 pad 7: Net-(U3-Pad7) -> Blanking
- U3 pad 8: Net-(U3-Pad8) -> pin2
- U3 pad 9: Net-(U3-Pad9) -> pin1
- X1 pad 1: Net-(X1-Pad1) -> +3V3
- X1 pad 2: Net-(X1-Pad2) -> GND
- X1 pad 3: Net-(X1-Pad3) -> clk_1M2
- X1 pad 4: Net-(X1-Pad4) -> +3V3
Routing:
- net +3V3: track 53.3 -> 80.4 mm, vias 8 -> 11
- net +5V: track 0.00 -> 22.3 mm
- net clk_1M2: track 0.00 -> 13.8 mm, vias 0 -> 2
- net GND: track 18.9 -> 31.4 mm, vias 14 -> 23
- net pin1: track 0.00 -> 10.5 mm, vias 0 -> 2
- net clk_100k: track 0.00 -> 9.48 mm
- net clk_80k: track 0.00 -> 8.44 mm
- net led: track 0.00 -> 8.32 mm
- net clk_60k: track 0.00 -> 8.09 mm
- net E1A: track 0.00 -> 7.56 mm
- net clk_40k: track 0.00 -> 7.55 mm
- net clk_20k: track 0.00 -> 6.34 mm
- net pin2: track 0.00 -> 6.27 mm
- net Blanking: track 0.00 -> 5.96 mm
- net E2B: track 0.00 -> 5.89 mm
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- added copper zone on B.Cu, net GND
Other:
- board outline added: 29.3 x 22.3 mm
- rule trace_min: 0.1524 -> 0.254
- board text added: "100k"
- board text added: "1M2"
- board text added: "20k"
- board text added: "40k"
- board text added: "5V"
- board text added: "60k"
- board text added: "80k"
- board text added: "Clock Gen"
- board text added: "DSC1001AE5 001.2000"
- board text added: "Enc1"
- board text added: "Enc2"
- board text added: "LCMXO2 256HC"
- board text added: "LED"
- board text added: "ON"
- board text added: "telec"
- board text added: "~RST"
